Commit message: change geometry of the urdf

File: urdf/create3.urdf.xacro (robot description, xacro)
@@ -104,5 +104,5 @@
   <!-- laser -->
   <xacro:laser gazebo="$(arg gazebo)" namespace="$(arg namespace)">
-    <origin xyz="-0.09 0 ${0.05 + base_link_z_offset}"/>
+    <origin xyz="0.075 -0.03 ${0.05 + base_link_z_offset}"/>
   </xacro:laser>
   <!-- <xacro:if value="${'$(arg gazebo)' == 'classic'}">
