Commit message: new higher res map

File: urdf/empty_belly.urdf (robot description, URDF)
Before this commit: robot my_robot, 4 links, 3 joints
Links:
- added link imu_link; visual cylinder length=0.02 radius=0.035
Joints:
- added joint imu_joint: type fixed, parent base_link, child imu_link, origin xyz=0.28 0 0.17 rpy=0 0 0
